File: layouts/thermocouple_v0.1.brd (EAGLE design)
At the start: 35 x 34 mm, 28 parts, among them J1 1X2-3.5MM, J2 1X2-3.5MM, J3 1X2-3.5MM, J4 1X2-3.5MM, U1 MAX31855, U2 MAX31855, U3 MAX31855, U4 MAX31855, U5 MAX8687

Commit message: fixed eagle errors due to upgrade to 6.5
Parts:
- U5: value MAX8687 -> MAX8867
Changed lines of the file:
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@@
 <?xml version="1.0" encoding="utf-8"?>
 <!DOCTYPE eagle SYSTEM "eagle.dtd">
-<eagle version="6.3">
+<eagle version="6.6.0">
 <drawing>
 <settings>
@@
 <layers>
 <layer number="1" name="Top" color="4" fill="1" visible="yes" active="yes"/>
-<layer number="2" name="Route2" color="1" fill="3" visible="no" active="no"/>
+<layer number="2" name="Route2" color="14" fill="3" visible="no" active="no"/>
 <layer number="3" name="Route3" color="4" fill="3" visible="no" active="no"/>
 <layer number="4" name="Route4" color="1" fill="4" visible="no" active="no"/>
@@
 <layer number="13" name="Route13" color="4" fill="5" visible="no" active="no"/>
 <layer number="14" name="Route14" color="1" fill="6" visible="no" active="no"/>
-<layer number="15" name="Route15" color="4" fill="6" visible="no" active="no"/>
+<layer number="15" name="Route15" color="10" fill="6" visible="no" active="no"/>
 <layer number="16" name="Bottom" color="1" fill="1" visible="yes" active="yes"/>
 <layer number="17" name="Pads" color="2" fill="1" visible="yes" active="yes"/>
@@
 <attribute name="NAME" x="10.905" y="25.079" size="0.8128" layer="25" ratio="10" rot="R180"/>
 </element>
-<element name="U5" library="maxim" package="SOT23-5L" value="MAX8687" x="3" y="25" smashed="yes">
+<element name="U5" library="maxim" package="SOT23-5L" value="MAX8867" x="3" y="25" smashed="yes">
 <attribute name="NAME" x="2.995" y="21.805" size="0.8128" layer="25"/>
 <attribute name="VALUE" x="1.095" y="21.825" size="1.27" layer="27"/>
