File: layouts/stm32f76XV_breakout.sch (EAGLE design)
At the start: 52 parts, among them J1 FTSH-105-01-F-DV-K, K1 USB-MICROZX62R-B, K2 MICRO_SD01, Q1 25 MHz, T2 FDC5614P, U3 LMZ21701, U5 NUF2221

Commit message: added triac driver board
Parts:
- added LED_DC: (no value), led:LEDCHIPLED_0603
- added R18: 4k7, rcl:R-EU_R0603
Connections:
- net N$23 renamed LMZ_VIN
- net N$5 renamed LMZ_SS
- net N$7 renamed LMZ_PG
- net N$8 renamed LMZ_FB
- net V_IN renamed SUPPLY
- new net N$5: LED_DC.A, R18.2
- net +3V3: now also R18.1
- net GND: now also LED_DC.C
